File: hardware/transmitter/Bluetrackr-transmitter.sch (KiCad schematic (older format))
At the start: 29 parts

Commit message: Remove pull down resistor on button
Parts:
- removed R?: R, symbol Device:R
Connections:
- wire segments 90 -> 89
Other:
- moved on the sheet: J?
Changed lines of the file:
@@
 Text GLabel 10100 1500 0    50   Input ~ 0
 MPU_CS
-Text GLabel 10100 1600 0    50   Input ~ 0
-MPU_FSYNC
 NoConn ~ 10100 1100
 NoConn ~ 10100 1200
@@
 L Connector:Conn_01x02_Female J?
 U 1 1 5DA77594
-P 10300 1950
-F 0 "J?" H 10350 1950 50  0000 L CNN
-F 1 "Battery_Connector" H 10350 1850 50  0000 L CNN
-F 2 "" H 10300 1950 50  0001 C CNN
-F 3 "~" H 10300 1950 50  0001 C CNN
-	1    10300 1950
+P 10300 2100
+F 0 "J?" H 10350 2100 50  0000 L CNN
+F 1 "Battery_Connector" H 10350 2000 50  0000 L CNN
+F 2 "" H 10300 2100 50  0001 C CNN
+F 3 "~" H 10300 2100 50  0001 C CNN
+	1    10300 2100
 	1    0    0    -1
 $EndComp
@@
 L power:+BATT #PWR?
 U 1 1 5DA78455
-P 10000 1950
-F 0 "#PWR?" H 10000 1800 50  0001 C CNN
-F 1 "+BATT" V 10015 2077 50  0000 L CNN
-F 2 "" H 10000 1950 50  0001 C CNN
-F 3 "" H 10000 1950 50  0001 C CNN
-	1    10000 1950
+P 10000 2100
+F 0 "#PWR?" H 10000 1950 50  0001 C CNN
+F 1 "+BATT" V 10015 2227 50  0000 L CNN
+F 2 "" H 10000 2100 50  0001 C CNN
+F 3 "" H 10000 2100 50  0001 C CNN
+	1    10000 2100
 	0    -1   -1   0
 $EndComp
@@
 L power:-BATT #PWR?
 U 1 1 5DA79547
-P 10000 2050
-F 0 "#PWR?" H 10000 1900 50  0001 C CNN
-F 1 "-BATT" V 10015 2177 50  0000 L CNN
-F 2 "" H 10000 2050 50  0001 C CNN
-F 3 "" H 10000 2050 50  0001 C CNN
-	1    10000 2050
+P 10000 2200
+F 0 "#PWR?" H 10000 2050 50  0001 C CNN
+F 1 "-BATT" V 10015 2327 50  0000 L CNN
+F 2 "" H 10000 2200 50  0001 C CNN
+F 3 "" H 10000 2200 50  0001 C CNN
+	1    10000 2200
 	0    -1   -1   0
 $EndComp
@@
 L power:-BATT #PWR?
 U 1 1 5DA84C45
-P 9100 1950
-F 0 "#PWR?" H 9100 1800 50  0001 C CNN
-F 1 "-BATT" V 9115 2077 50  0000 L CNN
-F 2 "" H 9100 1950 50  0001 C CNN
-F 3 "" H 9100 1950 50  0001 C CNN
-	1    9100 1950
+P 9100 2100
+F 0 "#PWR?" H 9100 1950 50  0001 C CNN
+F 1 "-BATT" V 9115 2227 50  0000 L CNN
+F 2 "" H 9100 2100 50  0001 C CNN
+F 3 "" H 9100 2100 50  0001 C CNN
+	1    9100 2100
 	0    -1   -1   0
 $EndComp
@@
 L power:GND #PWR?
 U 1 1 5DA864FF
-P 9200 2050
-F 0 "#PWR?" H 9200 1800 50  0001 C CNN
-F 1 "GND" H 9205 1877 50  0000 C CNN
-F 2 "" H 9200 2050 50  0001 C CNN
-F 3 "" H 9200 2050 50  0001 C CNN
-	1    9200 2050
-	1    0    0    -1
-$EndComp
-Wire Wire Line
-	10000 1950 10100 1950
-Wire Wire Line
-	10100 2050 10000 2050
-Wire Wire Line
-	9100 1950 9200 1950
-Wire Wire Line
-	9200 1950 9200 2050
+P 9200 2200
+F 0 "#PWR?" H 9200 1950 50  0001 C CNN
+F 1 "GND" H 9205 2027 50  0000 C CNN
+F 2 "" H 9200 2200 50  0001 C CNN
+F 3 "" H 9200 2200 50  0001 C CNN
+	1    9200 2200
+	1    0    0    -1
+$EndComp
+Wire Wire Line
+	10000 2100 10100 2100
+Wire Wire Line
+	10100 2200 10000 2200
+Wire Wire Line
+	9100 2100 9200 2100
+Wire Wire Line
+	9200 2100 9200 2200
 $Comp
 L Device:R R?
@@
 $EndComp
 $Comp
-L power:GND #PWR?
-U 1 1 5DAD2127
-P 4950 1700
-F 0 "#PWR?" H 4950 1450 50  0001 C CNN
-F 1 "GND" H 4955 1527 50  0000 C CNN
-F 2 "" H 4950 1700 50  0001 C CNN
-F 3 "" H 4950 1700 50  0001 C CNN
-	1    4950 1700
-	1    0    0    -1
-$EndComp
-$Comp
 L power:+3V3 #PWR?
 U 1 1 5DAD2A53
@@
 	1    0    0    -1
 $EndComp
-$Comp
-L Device:R R?
-U 1 1 5DAD32E9
-P 4950 1450
-F 0 "R?" H 5020 1496 50  0000 L CNN
-F 1 "R" H 5020 1405 50  0000 L CNN
-F 2 "" V 4880 1450 50  0001 C CNN
-F 3 "~" H 4950 1450 50  0001 C CNN
-	1    4950 1450
-	1    0    0    -1
-$EndComp
 Wire Wire Line
 	5450 1200 5550 1200
-Text GLabel 4850 1200 0    50   Input ~ 0
+Text GLabel 4950 1200 0    50   Input ~ 0
 BTN_PAIR
-Wire Wire Line
-	4850 1200 4950 1200
-Wire Wire Line
-	4950 1700 4950 1600
-Wire Wire Line
-	4950 1300 4950 1200
-Connection ~ 4950 1200
-Wire Wire Line
-	4950 1200 5050 1200
 Wire Wire Line
 	5550 1100 5550 1200
@@
 Text GLabel 6150 4050 2    50   Input ~ 0
 LED_POWER
+$Comp
+L power:GND #PWR?
+U 1 1 5DA98822
+P 10000 1700
+F 0 "#PWR?" H 10000 1450 50  0001 C CNN
+F 1 "GND" H 10005 1527 50  0000 C CNN
+F 2 "" H 10000 1700 50  0001 C CNN
+F 3 "" H 10000 1700 50  0001 C CNN
+	1    10000 1700
+	1    0    0    -1
+$EndComp
+Wire Wire Line
+	10000 1700 10000 1600
+Wire Wire Line
+	10000 1600 10100 1600
+Wire Wire Line
+	4950 1200 5050 1200
 $EndSCHEMATC

Commit message: Finish transmitter schematic, pass DRC
Parts:
- removed J?: MPU9250_Connector, symbol Connector:Conn_01x10_Female
- removed TP?: Reset, symbol Connector:TestPoint
- added M2: MPU-9250, symbol Modules:MPU-9250
- added R5: 10k, symbol Device:R
- added SW1: Button_Reset, symbol Switch:SW_Push
- gave numbers to parts that had none: 26
Connections:
- net labels removed: MPU_FSYNC, NRST
- wire segments 89 -> 95
- no-connect marks 5 -> 28
Other:
- moved on the sheet: C7, J1, J2

Commit message: Layout the transmitter pcb
Parts:
- C1, C2, C3, C4, C5, C6, C7: footprint (none) -> Capacitor_SMD:C_0805_2012Metric_Pad1.15x1.40mm_HandSolder
- C8: footprint (none) -> Capacitor_SMD:C_1206_3216Metric_Pad1.42x1.75mm_HandSolder
- D1: value LED -> STATUS_LED; footprint (none) -> LED_SMD:LED_1206_3216Metric_Pad1.42x1.75mm_HandSolder
- D2: value LED -> POWER_LED; footprint (none) -> LED_SMD:LED_1206_3216Metric_Pad1.42x1.75mm_HandSolder
- H1, H2, H3, H4: footprint (none) -> MountingHole:MountingHole_2.2mm_M2
- J1: footprint (none) -> Connector_PinHeader_2.54mm:PinHeader_1x04_P2.54mm_Vertical
- J2: footprint (none) -> Connector_PinHeader_2.54mm:PinHeader_1x02_P2.54mm_Vertical
- M1: footprint (none) -> Modules:TP4056
- M2: footprint (none) -> Modules:Module_10pin_15x26mm
- R1, R2, R3, R4, R5, R6: footprint (none) -> Resistor_SMD:R_0805_2012Metric_Pad1.15x1.40mm_HandSolder
- SW1: footprint (none) -> Button_Switch_THT:SW_PUSH_6mm_H4.3mm
- SW2: footprint (none) -> Button_Switch_THT:SW_PUSH_6mm_H9.5mm
Connections:
- net labels removed: MPU_GND, MPU_VCC
- wire segments 95 -> 93
Other:
- moved on the sheet: D2, R2
