File: hardware/transmitter/Bluetrackr-transmitter.sch (KiCad schematic (older format))
At the start: 29 parts, among them J1 Programming_Connector, J2 Battery_Connector, M1 TP4056, M2 MPU-9250, SW1 Button_Reset, SW2 SW_Pair, U1 MIC5205-3.3YM5, U2 STM32F103C8Tx, U3 NRF24L01_Breakout

Commit message: Replace global labels with net labels
Connections:
- net labels added: NRF_CSN
- net labels removed: NRF_CS
- no-connect marks 28 -> 27
Other:
- note removed: "no power from\nprogramming"
Changed lines of the file:
@@
 Sheet 1 1
 Title "Bluetrackr-transmitter"
-Date ""
-Rev ""
+Date "2019-11-24"
+Rev "2"
 Comp ""
 Comment1 ""
@@
 Wire Wire Line
 	4600 2850 4850 2850
-Text GLabel 6150 5150 2    50   Input ~ 0
-SWCLK
-Text GLabel 6150 5050 2    50   Input ~ 0
-SWDIO
-Text GLabel 9700 1700 0    50   Input ~ 0
-MPU_INT
-Text GLabel 9700 1800 0    50   Input ~ 0
-MPU_CS
 NoConn ~ 9700 1400
 NoConn ~ 9700 1500
@@
 	1    0    0    -1
 $EndComp
-Text GLabel 4850 4850 0    50   Input ~ 0
-MPU_INT
-Text GLabel 4850 3750 0    50   Input ~ 0
-MPU_CS
 $Comp
 L Regulator_Linear:MIC5205-3.3YM5 U1
@@
 Wire Wire Line
 	1950 1400 1700 1400
-Text Notes 750  900  0    118  ~ 0
+Text Notes 950  900  0    79   ~ 16
 3.3V REGULATOR
 $Comp
@@
 	1    0    0    -1
 $EndComp
-Text GLabel 3650 1200 2    50   Input ~ 0
-VBAT_SENSE
-Text GLabel 6150 3750 2    50   Input ~ 0
-VBAT_SENSE
 $Comp
 L power:+BATT #PWR0122
@@
 Wire Wire Line
 	5450 1200 5550 1200
-Text GLabel 4950 1200 0    50   Input ~ 0
-BTN_PAIR
 Wire Wire Line
 	5550 1100 5550 1200
-Text GLabel 4850 4550 0    50   Input ~ 0
-BTN_PAIR
 $Comp
 L RF:NRF24L01_Breakout U3
@@
 	1    0    0    -1
 $EndComp
-Text GLabel 9400 5350 0    50   Input ~ 0
-NRF_CS
-Text GLabel 9400 5550 0    50   Input ~ 0
-NRF_CE
-Text GLabel 4850 3850 0    50   Input ~ 0
-NRF_CS
-Text GLabel 4850 4250 0    50   Input ~ 0
-NRF_CE
-Text GLabel 4850 4750 0    50   Input ~ 0
-NRF_INT
-Text GLabel 6150 4450 2    50   Input ~ 0
-SPI_MOSI
-Text GLabel 6150 4350 2    50   Input ~ 0
-SPI_MISO
-Text GLabel 6150 4250 2    50   Input ~ 0
-SPI_SCK
-Text GLabel 9400 5050 0    50   Input ~ 0
-SPI_MOSI
-Text GLabel 9400 5150 0    50   Input ~ 0
-SPI_MISO
-Text GLabel 9400 5250 0    50   Input ~ 0
-SPI_SCK
-Text GLabel 9700 1200 0    50   Input ~ 0
-SPI_SCK
-Text GLabel 9700 1300 0    50   Input ~ 0
-SPI_MOSI
-Text GLabel 9700 1600 0    50   Input ~ 0
-SPI_MISO
-Text GLabel 9400 5650 0    50   Input ~ 0
-NRF_INT
 $Comp
 L Device:C C8
@@
 	1    0    0    -1
 $EndComp
-Text GLabel 7000 1300 2    50   Input ~ 0
-SWCLK
-Text GLabel 7000 1100 2    50   Input ~ 0
-SWDIO
 $Comp
 L power:GND #PWR0129
@@
 Wire Wire Line
 	7400 1200 7400 1300
-NoConn ~ 7000 1400
-Text Notes 6700 1600 0    50   ~ 0
-no power from\nprogramming
 $Comp
 L Mechanical:MountingHole H4
@@
 Wire Wire Line
 	1400 3800 1400 3900
-Text GLabel 1400 3000 1    50   Input ~ 0
-LED_STATUS
-Text GLabel 1800 3000 1    50   Input ~ 0
-LED_POWER
 $Comp
 L Device:R R2
@@
 Wire Wire Line
 	1400 3100 1400 3000
-Text GLabel 6150 3950 2    50   Input ~ 0
-LED_STATUS
-Text GLabel 6150 4050 2    50   Input ~ 0
-LED_POWER
 $Comp
 L power:GND #PWR0132
@@
 	9150 1100 9700 1100
 Connection ~ 5350 2350
+Text Label 7000 1100 0    50   ~ 0
+SWDIO
+Text Label 7000 1300 0    50   ~ 0
+SWCLK
+Text Label 6150 5050 0    50   ~ 0
+SWDIO
+Text Label 6150 5150 0    50   ~ 0
+SWCLK
+Text Label 6150 3750 0    50   ~ 0
+VBAT_SENSE
+Text Label 6150 3950 0    50   ~ 0
+LED_STATUS
+Text Label 6150 4050 0    50   ~ 0
+LED_POWER
+Text Label 6150 4250 0    50   ~ 0
+SPI_SCK
+Text Label 6150 4350 0    50   ~ 0
+SPI_MISO
+Text Label 6150 4450 0    50   ~ 0
+SPI_MOSI
+Text Label 4850 3750 2    50   ~ 0
+MPU_CS
+Text Label 4850 3850 2    50   ~ 0
+NRF_CSN
+Text Label 4850 4250 2    50   ~ 0
+NRF_CE
+Text Label 4850 4550 2    50   ~ 0
+BTN_PAIR
+Text Label 4850 4750 2    50   ~ 0
+NRF_INT
+Text Label 4850 4850 2    50   ~ 0
+MPU_INT
+Text Label 1400 3000 1    50   ~ 0
+LED_STATUS
+Text Label 1800 3000 1    50   ~ 0
+LED_POWER
+Text Label 3650 1200 0    50   ~ 0
+VBAT_SENSE
+Text Label 4950 1200 2    50   ~ 0
+BTN_PAIR
+Text Label 9700 1200 2    50   ~ 0
+SPI_SCK
+Text Label 9700 1300 2    50   ~ 0
+SPI_MOSI
+Text Label 9700 1600 2    50   ~ 0
+SPI_MISO
+Text Label 9700 1700 2    50   ~ 0
+MPU_INT
+Text Label 9700 1800 2    50   ~ 0
+MPU_CS
+Text Label 9400 5250 2    50   ~ 0
+SPI_SCK
+Text Label 9400 5350 2    50   ~ 0
+NRF_CSN
+Text Label 9400 5150 2    50   ~ 0
+SPI_MISO
+Text Label 9400 5050 2    50   ~ 0
+SPI_MOSI
+Text Label 9400 5550 2    50   ~ 0
+NRF_CE
+Text Label 9400 5650 2    50   ~ 0
+NRF_INT
 $EndSCHEMATC
